File: Panel/mikrokosmos_panel.kicad_pcb (KiCad board)
At the start: 2 copper layers, 200 x 25 mm, 10 parts

Commit message: Update .gitignore, Gerbers
Other:
- board text added: "JLCJLCJLCJLC"
- board text added: "Panel design by Rich Holmes Apr 2020"
